File: hub.kicad_sch (KiCad schematic)
At the start: 38 parts, among them IC1 48MHz, IC3 TUSB2036VF, J10 USB_C_Receptacle_USB2.0, J6 USB_A, J7 USB_A

Commit message: Update to KiCad 8.
Parts:
- renumbered D1 to D3
