File: openkayo.kicad_pcb (KiCad board)
At the start: 2 copper layers, 80 x 70 mm, 82 parts, among them IC1 48MHz, IC2 TCAN332, IC3 TUSB2036VF, J1 Conn_01x03_Socket, J10 USB_C_Receptacle_USB2.0, J2 CAN_TERM, J3 CAN_BUS, J5 Conn_01x02, J6 USB_A, J7 USB_A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

Commit message: Added footprint for ESP32-S3-WROOM-1.  Aligned in schematic.
Routing:
- net unconnected-(J10-SHIELD-PadS1)_1: track 21.9 -> 0.00 mm
- net unconnected-(J10-SHIELD-PadS1): track 0.00 -> 21.9 mm
